File: 8bit-decoder-visualizer.kicad_pcb (KiCad board)
At the start: 2 copper layers, 63.5 x 85.1 mm, 45 parts, among them SW1 SW_SPDT, SW2 SW_SPDT, SW3 SW_SPDT, SW4 SW_SPDT, SW5 SW_SPDT, SW6 SW_SPDT, SW7 SW_SPDT, SW8 SW_SPDT, U1 LED Display Module, U2 LED Display Module, U3 LED Display Module, U4 LED Display Module, U5 LED Display Module, U6 LED Display Module, U7 74HC595, U8 XIAO_General

Commit message: 配置配線を調整して基板を小型化
Parts:
- moved R8 48.9 mm to (134.0, 83.8), turned to 0 degrees
- moved R7 41.1 mm to (134.0, 86.4), turned to 0 degrees
- moved R6 33.3 mm to (134.0, 88.9), turned to 0 degrees
- moved R5 25.7 mm to (134.0, 91.4), turned to 0 degrees
- moved R4 18.5 mm to (134.0, 94.0), turned to 0 degrees
- moved R3 12.3 mm to (134.0, 96.5), turned to 0 degrees
- moved R1 5.12 mm to (120.7, 103.5)
- moved R2 5.12 mm to (128.3, 103.5)
- moved U7 2.56 mm to (130.8, 99.1)
- moved SW1 2.54 mm to (120.7, 122.0)
- moved SW2 2.54 mm to (128.3, 122.0)
- moved SW3 2.54 mm to (135.9, 122.0)
- moved SW4 2.54 mm to (143.5, 122.0)
- moved SW5 2.54 mm to (151.1, 122.0)
- moved SW6 2.54 mm to (158.8, 122.0)
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Routing:
- net Net-(U7-QH): track 66.1 -> 2.35 mm
- net Net-(D8-A): track 4.78 -> 59.6 mm
- net Net-(U7-QG): track 56.4 -> 2.35 mm
- net Net-(D7-A): track 4.78 -> 49.9 mm
- net Net-(U7-QF): track 46.7 -> 2.35 mm
- net Net-(D6-A): track 4.78 -> 40.2 mm
- net Net-(U7-QE): track 37.0 -> 2.35 mm
- net Net-(D5-A): track 4.78 -> 30.5 mm
- net Net-(U7-QD): track 27.3 -> 2.35 mm
- net Net-(D4-A): track 4.78 -> 20.8 mm
- net Net-(U7-QC): track 17.5 -> 2.35 mm
- net Net-(D3-A): track 4.78 -> 13.1 mm
- net Net-(U7-QA): track 14.2 -> 7.21 mm
- net Net-(U7-QB): track 10.6 -> 4.69 mm
- net /LED_CLK: track 154.0 -> 158.3 mm
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Other:
- board size 63.5 x 85.1 mm -> 63.5 x 82.6 mm
