File: rev2/rev2.kicad_pcb (KiCad board)
At the start: 2 copper layers, 118 parts, among them J1 USB_C_Receptacle_USB2.0_14P, Q1 BSS138, Q10 BSS138, Q11 BSS138, Q12 BSS138, Q13 BSS138, Q14 BSS138, Q15 BSS138, Q16 BSS138, Q2 BSS138, Q3 BSS138, Q4 BSS138, Q5 BSS138, Q6 BSS138, Q7 BSS138, Q8 BSS138, Q9 BSS138, SW1 SW_Push, SW2 SW_Push, SW3 SW_Push, SW4 SW_Push, SW5 SW_Push, SW6 SW_Push, SW7 SW_Push, SW8 SW_Push, U1 CH340N, U2 ATtiny1604-SS, U3 74HC595, U4 74HC595, U5 74HC595, U6 74HC595

Commit message: 回路図で消した部品を削除
Parts:
- removed Q1, Q10, Q11, Q12, Q13, Q14, Q15, Q16, Q2, Q3, Q4, Q5, Q6, Q7, Q8, Q9: BSS138, Package_TO_SOT_SMD:SOT-23
- removed R21, R22, R23, R24, R25, R26, R27, R28, R29, R30, R31, R32, R33, R34, R35, R36: 100R, Resistor_SMD:R_0603_1608Metric
- removed R37, R38, R39, R40, R41, R42, R43, R44, R45, R46, R47, R48, R49, R50, R51, R52: 10k, Resistor_SMD:R_0603_1608Metric
- moved U5 77.2 mm to (186.0, 105.8)
- moved U6 77.2 mm to (190.0, 105.8)
